File: discharge-board/CTRL-MINI-ED/regulator_3v3.kicad_sch (KiCad schematic)
At the start: 3 parts, among them U8 BD33FC0FP

Commit message: Add netlist class
Parts:
- renumbered C39 to C36, C40 to C37, U8 to U7
Changed lines of the file:
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@@
 	)
 	(hierarchical_label "VIN"
-		(shape passive)
+		(shape input)
 		(at 67.31 54.61 180)
 		(fields_autoplaced yes)
@@
 		(dnp no)
 		(fields_autoplaced yes)
-		(property "Reference" "#PWR057"
+		(property "Reference" "#PWR051"
 			(at 87.63 73.66 0)
 			(effects
@@
 			(project "CTRL-MINI-ED"
 				(path "/3fa1ca74-4d0d-40dd-8b5c-0d4be11bd5b5/a9794609-42db-49f0-aeeb-4c313a94f296"
-					(reference "#PWR057")
+					(reference "#PWR051")
 					(unit 1)
 				)
@@
 		(dnp no)
 		(fields_autoplaced yes)
-		(property "Reference" "U8"
+		(property "Reference" "U7"
 			(at 87.63 48.26 0)
 			(effects
@@
 			(project ""
 				(path "/3fa1ca74-4d0d-40dd-8b5c-0d4be11bd5b5/a9794609-42db-49f0-aeeb-4c313a94f296"
-					(reference "U8")
+					(reference "U7")
 					(unit 1)
 				)
@@
 		(on_board yes)
 		(dnp no)
-		(property "Reference" "C39"
+		(property "Reference" "C36"
 			(at 75.946 59.944 0)
 			(effects
@@
 			(project "CTRL-MINI-ED"
 				(path "/3fa1ca74-4d0d-40dd-8b5c-0d4be11bd5b5/a9794609-42db-49f0-aeeb-4c313a94f296"
-					(reference "C39")
+					(reference "C36")
 					(unit 1)
 				)
@@
 		(on_board yes)
 		(dnp no)
-		(property "Reference" "C40"
+		(property "Reference" "C37"
 			(at 102.616 59.944 0)
 			(effects
@@
 			(project "CTRL-MINI-ED"
 				(path "/3fa1ca74-4d0d-40dd-8b5c-0d4be11bd5b5/a9794609-42db-49f0-aeeb-4c313a94f296"
-					(reference "C40")
+					(reference "C37")
 					(unit 1)
 				)
