File: discharge-board/CTRL-MINI-ED/relay_half_bridge.kicad_sch (KiCad schematic)
At the start: 10 parts, among them K1 G2RL-1A-E, K2 G2RL-1A-E, Q1 Q_NMOS_GSD, Q2 Q_NMOS_GSD

Commit message: Add netlist class
Parts:
- renumbered R12 to R10, R13 to R11, R10 to R8, R11 to R9
Connections:
- net L_COIL-: now reaches D4.2 (A), K2.A2, Q2.3 (D)
- net H_COIL-: now reaches D3.2 (A), K1.A1, Q1.3 (D)
Changed lines of the file:
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@@
+		)
+	)
+	(label "H_COIL-"
+		(at 97.79 57.15 0)
+		(fields_autoplaced yes)
+		(effects
+			(font
+				(size 1.27 1.27)
+			)
+			(justify left bottom)
+		)
+	)
+	(label "L_COIL-"
+		(at 97.79 114.3 0)
+		(fields_autoplaced yes)
+		(effects
+			(font
+				(size 1.27 1.27)
+			)
+			(justify left bottom)
 		)
 	)
@@
 		(on_board yes)
 		(dnp no)
-		(property "Reference" "R13"
+		(property "Reference" "R11"
 			(at 92.71 133.35 0)
 			(effects
@@
 			(project "CTRL-MINI-ED"
 				(path "/3fa1ca74-4d0d-40dd-8b5c-0d4be11bd5b5/61d269a5-db7e-4708-be89-e9446bc418aa"
-					(reference "R13")
+					(reference "R11")
 					(unit 1)
 				)
 				(path "/3fa1ca74-4d0d-40dd-8b5c-0d4be11bd5b5/6c946658-61d5-4fe0-8cd3-b855580e1af0"
-					(reference "R17")
+					(reference "R15")
 					(unit 1)
 				)
 				(path "/3fa1ca74-4d0d-40dd-8b5c-0d4be11bd5b5/701333a2-35b5-41e7-9f83-3a206a1cf781"
-					(reference "R21")
+					(reference "R19")
 					(unit 1)
 				)
@@
 		(on_board yes)
 		(dnp no)
-		(property "Reference" "#PWR019"
+		(property "Reference" "#PWR013"
 			(at 106.68 39.37 0)
 			(effects
@@
 			(project "CTRL-MINI-ED"
 				(path "/3fa1ca74-4d0d-40dd-8b5c-0d4be11bd5b5/61d269a5-db7e-4708-be89-e9446bc418aa"
-					(reference "#PWR019")
+					(reference "#PWR013")
 					(unit 1)
 				)
 				(path "/3fa1ca74-4d0d-40dd-8b5c-0d4be11bd5b5/6c946658-61d5-4fe0-8cd3-b855580e1af0"
-					(reference "#PWR023")
+					(reference "#PWR017")
 					(unit 1)
 				)
 				(path "/3fa1ca74-4d0d-40dd-8b5c-0d4be11bd5b5/701333a2-35b5-41e7-9f83-3a206a1cf781"
-					(reference "#PWR027")
+					(reference "#PWR021")
 					(unit 1)
 				)
@@
 		(on_board yes)
 		(dnp no)
-		(property "Reference" "R12"
+		(property "Reference" "R10"
 			(at 90.17 123.698 90)
 			(effects
@@
 			(project "CTRL-MINI-ED"
 				(path "/3fa1ca74-4d0d-40dd-8b5c-0d4be11bd5b5/61d269a5-db7e-4708-be89-e9446bc418aa"
-					(reference "R12")
+					(reference "R10")
 					(unit 1)
 				)
 				(path "/3fa1ca74-4d0d-40dd-8b5c-0d4be11bd5b5/6c946658-61d5-4fe0-8cd3-b855580e1af0"
-					(reference "R16")
+					(reference "R14")
 					(unit 1)
 				)
 				(path "/3fa1ca74-4d0d-40dd-8b5c-0d4be11bd5b5/701333a2-35b5-41e7-9f83-3a206a1cf781"
-					(reference "R20")
+					(reference "R18")
 					(unit 1)
 				)
@@
 		(on_board yes)
 		(dnp no)
-		(property "Reference" "R11"
+		(property "Reference" "R9"
 			(at 92.964 69.088 0)
 			(effects
@@
 			(project "CTRL-MINI-ED"
 				(path "/3fa1ca74-4d0d-40dd-8b5c-0d4be11bd5b5/61d269a5-db7e-4708-be89-e9446bc418aa"
-					(reference "R11")
+					(reference "R9")
 					(unit 1)
 				)
 				(path "/3fa1ca74-4d0d-40dd-8b5c-0d4be11bd5b5/6c946658-61d5-4fe0-8cd3-b855580e1af0"
-					(reference "R15")
+					(reference "R13")
 					(unit 1)
 				)
 				(path "/3fa1ca74-4d0d-40dd-8b5c-0d4be11bd5b5/701333a2-35b5-41e7-9f83-3a206a1cf781"
-					(reference "R19")
+					(reference "R17")
 					(unit 1)
 				)
@@
 		(on_board yes)
 		(dnp no)
-		(property "Reference" "#PWR020"
+		(property "Reference" "#PWR014"
 			(at 106.68 83.82 0)
 			(effects
@@
 			(project "CTRL-MINI-ED"
 				(path "/3fa1ca74-4d0d-40dd-8b5c-0d4be11bd5b5/61d269a5-db7e-4708-be89-e9446bc418aa"
-					(reference "#PWR020")
+					(reference "#PWR014")
 					(unit 1)
 				)
 				(path "/3fa1ca74-4d0d-40dd-8b5c-0d4be11bd5b5/6c946658-61d5-4fe0-8cd3-b855580e1af0"
-					(reference "#PWR024")
+					(reference "#PWR018")
 					(unit 1)
 				)
 				(path "/3fa1ca74-4d0d-40dd-8b5c-0d4be11bd5b5/701333a2-35b5-41e7-9f83-3a206a1cf781"
-					(reference "#PWR028")
+					(reference "#PWR022")
 					(unit 1)
 				)
@@
 		(on_board yes)
 		(dnp no)
-		(property "Reference" "#PWR021"
+		(property "Reference" "#PWR015"
 			(at 106.68 96.52 0)
 			(effects
@@
 			(project "CTRL-MINI-ED"
 				(path "/3fa1ca74-4d0d-40dd-8b5c-0d4be11bd5b5/61d269a5-db7e-4708-be89-e9446bc418aa"
-					(reference "#PWR021")
+					(reference "#PWR015")
 					(unit 1)
 				)
 				(path "/3fa1ca74-4d0d-40dd-8b5c-0d4be11bd5b5/6c946658-61d5-4fe0-8cd3-b855580e1af0"
-					(reference "#PWR025")
+					(reference "#PWR019")
 					(unit 1)
 				)
 				(path "/3fa1ca74-4d0d-40dd-8b5c-0d4be11bd5b5/701333a2-35b5-41e7-9f83-3a206a1cf781"
-					(reference "#PWR029")
+					(reference "#PWR023")
 					(unit 1)
 				)
@@
 		(on_board yes)
 		(dnp no)
-		(property "Reference" "#PWR022"
+		(property "Reference" "#PWR016"
 			(at 106.68 147.32 0)
 			(effects
@@
 			(project "CTRL-MINI-ED"
 				(path "/3fa1ca74-4d0d-40dd-8b5c-0d4be11bd5b5/61d269a5-db7e-4708-be89-e9446bc418aa"
-					(reference "#PWR022")
+					(reference "#PWR016")
 					(unit 1)
 				)
 				(path "/3fa1ca74-4d0d-40dd-8b5c-0d4be11bd5b5/6c946658-61d5-4fe0-8cd3-b855580e1af0"
-					(reference "#PWR026")
+					(reference "#PWR020")
 					(unit 1)
 				)
 				(path "/3fa1ca74-4d0d-40dd-8b5c-0d4be11bd5b5/701333a2-35b5-41e7-9f83-3a206a1cf781"
-					(reference "#PWR030")
+					(reference "#PWR024")
 					(unit 1)
 				)
@@
 		(on_board yes)
 		(dnp no)
-		(property "Reference" "R10"
+		(property "Reference" "R8"
 			(at 90.17 60.198 90)
 			(effects
@@
 			(project "CTRL-MINI-ED"
 				(path "/3fa1ca74-4d0d-40dd-8b5c-0d4be11bd5b5/61d269a5-db7e-4708-be89-e9446bc418aa"
-					(reference "R10")
+					(reference "R8")
 					(unit 1)
 				)
 				(path "/3fa1ca74-4d0d-40dd-8b5c-0d4be11bd5b5/6c946658-61d5-4fe0-8cd3-b855580e1af0"
-					(reference "R14")
+					(reference "R12")
 					(unit 1)
 				)
 				(path "/3fa1ca74-4d0d-40dd-8b5c-0d4be11bd5b5/701333a2-35b5-41e7-9f83-3a206a1cf781"
-					(reference "R18")
-					(unit 1)
-				)
+					(reference "R16")
+					(unit 1)
+				)

Commit message: Draft of PCB layout
Parts:
- removed K1, K2: G2RL-1A-E, Relay_THT:Relay_SPST_Omron_G2RL-1A-E, symbol Relay:G2RL-1A-E
- added K1, K3: G2RL-2, Relay_THT:Relay_DPDT_Omron_G2RL-2, symbol Relay:G2RL-2
Connections:
- net V+: now also K1.21
- net V-: now also K1.11
- net VRELAY: now also K1.A1, K3.A1
- net EN_H renamed SEL
- net EN_L renamed POL
- net H_COIL- renamed P_COIL-
- net P_COIL-: now also Q2.3 (D), K1.A2; no longer Q1.3 (D)
- net L_COIL- renamed S_COIL-
- net S_COIL-: now also Q1.3 (D), K3.A2; no longer Q2.3 (D)
- new net: K1.14, K1.22, K3.11, K3.21
- new net VOUT_0: K3.12, K3.22
- new net VOUT_1: K3.14, K3.24
- new net VOUT_COM: K1.12, K1.24
Other:
- note added: "SPEC POL=L, SEL=L: VOUT_COM=-, VOUT_0=+ (VOUT_1=HZ) POL=L, SEL=H: VOUT_COM=-, VOUT_1=+ (VOUT_0=HZ) POL=H, SEL=L: VOUT_COM=+, VOUT_0=- (VOUT_1=HZ) POL=H: SEL=H: VOUT_COM=+, VOUT_1=- (VOUT_0=HZ) VOUTs are also HZ during change in POL and/or SEL"
- note added: "VRELAY (24V) current draw max: 35mA"
- note removed: "VRELAY (24V) current draw max: 20mA (at most single relay active)"
