File: discharge-board/CTRL-MINI-ED/rp2040.kicad_sch (KiCad schematic)
At the start: 19 parts, among them U5 RP2040, U6 W25Q128JVS, Y1 12MHz

Commit message: Add netlist class
Parts:
- renumbered C23 to C20, C24 to C21, C25 to C22, C26 to C23, C27 to C24, C28 to C25, C29 to C26, C30 to C27, C31 to C28, C32 to C29, C33 to C30, C34 to C31, C35 to C32, C36 to C33, R32 to R30, R33 to R31, U5 to U4, U6 to U5

Commit message: Draft of PCB layout
Parts:
- added JP5: Jumper_2_Small_Bridged, Jumper:SolderJumper-2_P1.3mm_Bridged_RoundedPad1.0x1.5mm, symbol Jumper:Jumper_2_Small_Bridged
- added TP34, TP36, TP46: TestPoint_Alt, TestPoint:TestPoint_Pad_2.0x2.0mm, symbol Connector:TestPoint_Alt
- added TP42: TestPoint, TestPoint:TestPoint_Pad_D1.5mm, symbol Connector:TestPoint
- renumbered R30 to R24, R31 to R25
Connections:
- net +1V1: now also TP42.1
- net VDIGITAL: now also JP5.1 (A)
- net at U4.26 (RUN): now also JP5.2 (B)
- net at U4.27 (GPIO16): now also TP36.1
- net at U4.39 (GPIO27_ADC1): now also TP46.1
- net at U4.8 (GPIO6): now also TP34.1
- net MUX_GH: no longer names the net of U4.15 (GPIO12)
- net MUX_GL: no longer names the net of U4.16 (GPIO13)
- net MUX_TH renamed MUX_POL
- net MUX_TL renamed MUX_WG
- net MUX_WH renamed MUX_EN
- net MUX_WL: no longer names the net of U4.14 (GPIO11)
- no-connect marks 3 -> 16
